File: UniversalControlPanel.kicad_sch (KiCad schematic)
At the start: 23 parts, among them J1 USB_B_Micro, J2 Conn_ARM_JTAG_SWD_10, J3 Conn_01x40, J4 Conn_02x03_Odd_Even, SW1 SW_Push, U1 LM78M05_TO252, U2 MAX14783ExS, U3 USBLC6-2SC6, U4 AMS1117-3.3, U6 ESP32-S2-WROOM-I

Commit message: some changes
Parts:
- added D2: LED, LED_SMD:LED_0603_1608Metric, symbol Device:LED
- added J5: Conn_01x02, Connector_JST:JST_XH_B2B-XH-A_1x02_P2.50mm_Vertical, symbol Connector_Generic:Conn_01x02
- added R8: 120, Resistor_SMD:R_0805_2012Metric_Pad1.20x1.40mm_HandSolder, symbol Device:R
- added R9: R, Resistor_SMD:R_0402_1005Metric, symbol Device:R
Connections:
- net at U2.6 (A): now also J5.2 (Pin_2), R8.2
- net at U2.7 (B): now also J5.1 (Pin_1), R8.1
Changed lines of the file:
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@@
   (junction (at 254 86.36) (diameter 0) (color 0 0 0 0)
   )
+  (junction (at 57.15 163.83) (diameter 0) (color 0 0 0 0)
+  )
   (junction (at 38.1 59.69) (diameter 0) (color 0 0 0 0)
   )
@@
   )
   (junction (at 254 88.9) (diameter 0) (color 0 0 0 0)
+  )
+  (junction (at 57.15 171.45) (diameter 0) (color 0 0 0 0)
   )
   (junction (at 254 93.98) (diameter 0) (color 0 0 0 0)
@@
     (stroke (width 0) (type default) (color 0 0 0 0))
   )
+  (wire (pts (xy 66.04 163.83) (xy 66.04 166.37))
+    (stroke (width 0) (type default) (color 0 0 0 0))
+  )
   (wire (pts (xy 254 99.06) (xy 254 101.6))
     (stroke (width 0) (type default) (color 0 0 0 0))
@@
     (stroke (width 0) (type default) (color 0 0 0 0))
   )
+  (wire (pts (xy 57.15 163.83) (xy 66.04 163.83))
+    (stroke (width 0) (type default) (color 0 0 0 0))
+  )
   (wire (pts (xy 254 119.38) (xy 254 121.92))
     (stroke (width 0) (type default) (color 0 0 0 0))
@@
     (stroke (width 0) (type default) (color 0 0 0 0))
   )
+  (wire (pts (xy 66.04 168.91) (xy 66.04 171.45))
+    (stroke (width 0) (type default) (color 0 0 0 0))
+  )
+  (wire (pts (xy 66.04 166.37) (xy 67.31 166.37))
+    (stroke (width 0) (type default) (color 0 0 0 0))
+  )
   (wire (pts (xy 242.57 63.5) (xy 257.81 63.5))
     (stroke (width 0) (type default) (color 0 0 0 0))
@@
     (stroke (width 0) (type default) (color 0 0 0 0))
   )
+  (wire (pts (xy 53.34 171.45) (xy 57.15 171.45))
+    (stroke (width 0) (type default) (color 0 0 0 0))
+  )
   (wire (pts (xy 41.91 88.9) (xy 44.45 88.9))
     (stroke (width 0) (type default) (color 0 0 0 0))
@@
     (stroke (width 0) (type default) (color 0 0 0 0))
   )
+  (wire (pts (xy 67.31 168.91) (xy 66.04 168.91))
+    (stroke (width 0) (type default) (color 0 0 0 0))
+  )
   (wire (pts (xy 254 124.46) (xy 257.81 124.46))
     (stroke (width 0) (type default) (color 0 0 0 0))
@@
     (stroke (width 0) (type default) (color 0 0 0 0))
   )
+  (wire (pts (xy 53.34 163.83) (xy 57.15 163.83))
+    (stroke (width 0) (type default) (color 0 0 0 0))
+  )
   (wire (pts (xy 120.65 66.04) (xy 130.81 66.04))
     (stroke (width 0) (type default) (color 0 0 0 0))
@@
   )
   (wire (pts (xy 242.57 66.04) (xy 257.81 66.04))
+    (stroke (width 0) (type default) (color 0 0 0 0))
+  )
+  (wire (pts (xy 57.15 171.45) (xy 66.04 171.45))
     (stroke (width 0) (type default) (color 0 0 0 0))
   )
@@
     (pin "1")
   )
+  (symbol (lib_id "Device:LED") (at 93.98 105.41 0) (unit 1)
+    (in_bom yes) (on_board yes) (fields_autoplaced)
+    (property "Reference" "D2" (id 0) (at 92.3925 99.06 0))
+    (property "Value" "LED" (id 1) (at 92.3925 101.6 0))
+    (property "Footprint" "LED_SMD:LED_0603_1608Metric" (id 2) (at 93.98 105.41 0)
+      (effects (font (size 1.27 1.27)) hide)
+    )
+    (property "Datasheet" "~" (id 3) (at 93.98 105.41 0)
+      (effects (font (size 1.27 1.27)) hide)
+    )
+    (property "LCSC" "C2286" (id 4) (at 93.98 105.41 0)
+      (effects (font (size 1.27 1.27)) hide)
+    )
+    (pin "1")
+    (pin "2")
+  )
   (symbol (lib_id "power:GND") (at 217.17 53.34 0) (unit 1)
     (in_bom yes) (on_board yes) (fields_autoplaced)
@@
     )
     (pin "1")
+  )
+  (symbol (lib_id "Device:R") (at 83.82 100.33 0) (unit 1)
+    (in_bom yes) (on_board yes) (fields_autoplaced)
+    (property "Reference" "R9" (id 0) (at 86.36 99.0599 0)
+      (effects (font (size 1.27 1.27)) (justify left))
+    )
+    (property "Value" "R" (id 1) (at 86.36 101.5999 0)
+      (effects (font (size 1.27 1.27)) (justify left))
+    )
+    (property "Footprint" "Resistor_SMD:R_0402_1005Metric" (id 2) (at 82.042 100.33 90)
+      (effects (font (size 1.27 1.27)) hide)
+    )
+    (property "Datasheet" "~" (id 3) (at 83.82 100.33 0)
+      (effects (font (size 1.27 1.27)) hide)
+    )
+    (pin "1")
+    (pin "2")
+  )
+  (symbol (lib_id "Connector_Generic:Conn_01x02") (at 72.39 166.37 0) (unit 1)
+    (in_bom yes) (on_board yes) (fields_autoplaced)
+    (property "Reference" "J5" (id 0) (at 74.93 166.3699 0)
+      (effects (font (size 1.27 1.27)) (justify left))
+    )
+    (property "Value" "Conn_01x02" (id 1) (at 74.93 168.9099 0)
+      (effects (font (size 1.27 1.27)) (justify left))
+    )
+    (property "Footprint" "Connector_JST:JST_XH_B2B-XH-A_1x02_P2.50mm_Vertical" (id 2) (at 72.39 166.37 0)
+      (effects (font (size 1.27 1.27)) hide)
+    )
+    (property "Datasheet" "~" (id 3) (at 72.39 166.37 0)
+      (effects (font (size 1.27 1.27)) hide)
+    )
+    (pin "1")
+    (pin "2")
   )
   (symbol (lib_id "power:GND") (at 220.98 153.67 0) (unit 1)
@@
     (pin "1")
   )
+  (symbol (lib_id "Device:R") (at 57.15 167.64 0) (unit 1)
+    (in_bom yes) (on_board yes) (fields_autoplaced)
+    (property "Reference" "R8" (id 0) (at 59.69 166.3699 0)
+      (effects (font (size 1.27 1.27)) (justify left))
+    )
+    (property "Value" "120" (id 1) (at 59.69 168.9099 0)
+      (effects (font (size 1.27 1.27)) (justify left))
+    )
+    (property "Footprint" "Resistor_SMD:R_0805_2012Metric_Pad1.20x1.40mm_HandSolder" (id 2) (at 55.372 167.64 90)
+      (effects (font (size 1.27 1.27)) hide)
+    )
+    (property "Datasheet" "~" (id 3) (at 57.15 167.64 0)
+      (effects (font (size 1.27 1.27)) hide)
+    )
+    (pin "1")
+    (pin "2")
+  )
   (symbol (lib_id "Regulator_Linear:LM78M05_TO252") (at 38.1 27.94 0) (unit 1)
     (in_bom yes) (on_board yes) (fields_autoplaced)
@@
       (reference "D1") (unit 1) (value "B5819W SL") (footprint "Diode_SMD:D_SOD-123")
     )
+    (path "/2828fc7e-8bff-4048-9818-789eee5ebf14"
+      (reference "D2") (unit 1) (value "LED") (footprint "LED_SMD:LED_0603_1608Metric")
+    )
     (path "/9e9a9c73-4b54-4e2e-be5b-f73fb6d96cb7"
       (reference "J1") (unit 1) (value "USB_B_Micro") (footprint "Connector_USB:USB_Mini-B_Tensility_54-00023_Vertical")
@@
       (reference "J4") (unit 1) (value "Conn_02x03_Odd_Even") (footprint "Connector_PinHeader_2.54mm:PinHeader_2x03_P2.54mm_Vertical")
     )
+    (path "/44520b3c-5b04-43b9-a30e-22180c4b99f4"
+      (reference "J5") (unit 1) (value "Conn_01x02") (footprint "Connector_JST:JST_XH_B2B-XH-A_1x02_P2.50mm_Vertical")
+    )
     (path "/f220d6a7-3170-4e04-8de6-2df0c3962fe0"
       (reference "R1") (unit 1) (value "10k") (footprint "Resistor_SMD:R_0402_1005Metric")
@@
       (reference "R7") (unit 1) (value "R") (footprint "Resistor_SMD:R_0402_1005Metric")
     )
+    (path "/db585110-1207-43ee-b01c-739dfd5f4452"
+      (reference "R8") (unit 1) (value "120") (footprint "Resistor_SMD:R_0805_2012Metric_Pad1.20x1.40mm_HandSolder")
+    )
+    (path "/345f5a55-a200-4388-bac3-15d4257e82dd"
+      (reference "R9") (unit 1) (value "R") (footprint "Resistor_SMD:R_0402_1005Metric")
+    )
     (path "/0e592cd4-1950-44ef-9727-8e526f4c4e12"

Commit message: replaced with TSR
Parts:
- removed C1: 10u, Capacitor_SMD:C_1206_3216Metric, symbol Device:C
- removed U1: LM78M05_TO252, Package_TO_SOT_SMD:TO-252-2, symbol Regulator_Linear:LM78M05_TO252
- added U1: TSR_1-2450, Converter_DCDC:Converter_DCDC_TRACO_TSR-1_THT, symbol Regulator_Switching:TSR_1-2450
Connections:
- net +24V: now also U1.1 (Vin)
- net +5V: now also U1.3 (Vout)
- net GND: now also U1.2 (GND)
Other:
- note removed: "1.3V drop.. not really great.."
- note removed: "50K/W at 6cm^2 copper"
Changed lines of the file:
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@@
   (junction (at 81.28 27.94) (diameter 0) (color 0 0 0 0)
-  )
-  (junction (at 22.86 27.94) (diameter 0) (color 0 0 0 0)
   )
   (junction (at 254 121.92) (diameter 0) (color 0 0 0 0)
@@
     (stroke (width 0) (type default) (color 0 0 0 0))
   )
+  (wire (pts (xy 48.26 27.94) (xy 54.61 27.94))
+    (stroke (width 0) (type default) (color 0 0 0 0))
+  )
   (wire (pts (xy 161.29 96.52) (xy 165.1 96.52))
     (stroke (width 0) (type default) (color 0 0 0 0))
@@
     (stroke (width 0) (type default) (color 0 0 0 0))
   )
+  (wire (pts (xy 22.86 27.94) (xy 27.94 27.94))
+    (stroke (width 0) (type default) (color 0 0 0 0))
+  )
   (wire (pts (xy 254 119.38) (xy 254 121.92))
     (stroke (width 0) (type default) (color 0 0 0 0))
@@
     (stroke (width 0) (type default) (color 0 0 0 0))
   )
-  (wire (pts (xy 45.72 27.94) (xy 54.61 27.94))
-    (stroke (width 0) (type default) (color 0 0 0 0))
-  )
   (wire (pts (xy 113.03 73.66) (xy 130.81 73.66))
     (stroke (width 0) (type default) (color 0 0 0 0))
@@
   )
   (wire (pts (xy 254 121.92) (xy 257.81 121.92))
-    (stroke (width 0) (type default) (color 0 0 0 0))
-  )
-  (wire (pts (xy 22.86 27.94) (xy 30.48 27.94))
     (stroke (width 0) (type default) (color 0 0 0 0))
   )
@@
     (effects (font (size 1.27 1.27)) (justify left bottom))
   )
-  (text "50K/W at 6cm^2 copper" (at 27.94 17.78 0)
-    (effects (font (size 1.27 1.27)) (justify left bottom))
-  )
   (text "perhaps a R (22E) and C to GND (22p)" (at 20.32 124.46 0)
     (effects (font (size 1.27 1.27)) (justify left bottom))
@@
   (text "4DLCD-24320240\nIL9341\nFT6236V\npin 1 is first from left from front"
     (at 245.11 48.26 0)
-    (effects (font (size 1.27 1.27)) (justify left bottom))
-  )
-  (text "1.3V drop.. not really great.." (at 63.5 17.78 0)
     (effects (font (size 1.27 1.27)) (justify left bottom))
   )
@@
     )
     (property "Datasheet" "" (id 3) (at 92.71 27.94 0)
-      (effects (font (size 1.27 1.27)) hide)
-    )
-    (pin "1")
-  )
-  (symbol (lib_id "power:GND") (at 22.86 35.56 0) (unit 1)
-    (in_bom yes) (on_board yes) (fields_autoplaced)
-    (property "Reference" "#PWR03" (id 0) (at 22.86 41.91 0)
-      (effects (font (size 1.27 1.27)) hide)
-    )
-    (property "Value" "GND" (id 1) (at 22.86 40.64 0))
-    (property "Footprint" "" (id 2) (at 22.86 35.56 0)
-      (effects (font (size 1.27 1.27)) hide)
-    )
-    (property "Datasheet" "" (id 3) (at 22.86 35.56 0)
       (effects (font (size 1.27 1.27)) hide)
     )
@@
     (pin "2")
   )
-  (symbol (lib_id "Regulator_Linear:LM78M05_TO252") (at 38.1 27.94 0) (unit 1)
-    (in_bom yes) (on_board yes) (fields_autoplaced)
-    (property "Reference" "U1" (id 0) (at 38.1 20.32 0))
-    (property "Value" "LM78M05_TO252" (id 1) (at 38.1 22.86 0))
-    (property "Footprint" "Package_TO_SOT_SMD:TO-252-2" (id 2) (at 38.1 22.225 0)
-      (effects (font (size 1.27 1.27) italic) hide)
-    )
-    (property "Datasheet" "https://www.onsemi.com/pub/Collateral/MC78M00-D.PDF" (id 3) (at 38.1 29.21 0)
-      (effects (font (size 1.27 1.27)) hide)
-    )
-    (pin "1")
-    (pin "2")
-    (pin "3")
-  )
   (symbol (lib_id "power:GND") (at 146.05 116.84 0) (unit 1)
     (in_bom yes) (on_board yes) (fields_autoplaced)
@@
     )
     (pin "1")
-  )
-  (symbol (lib_id "Device:C") (at 22.86 31.75 0) (unit 1)
-    (in_bom yes) (on_board yes) (fields_autoplaced)
-    (property "Reference" "C1" (id 0) (at 26.67 30.4799 0)
-      (effects (font (size 1.27 1.27)) (justify left))
-    )
-    (property "Value" "10u" (id 1) (at 26.67 33.0199 0)
-      (effects (font (size 1.27 1.27)) (justify left))
-    )
-    (property "Footprint" "Capacitor_SMD:C_1206_3216Metric" (id 2) (at 23.8252 35.56 0)
-      (effects (font (size 1.27 1.27)) hide)
-    )
-    (property "Datasheet" "~" (id 3) (at 22.86 31.75 0)
-      (effects (font (size 1.27 1.27)) hide)
-    )
-    (property "LCSC" "C13585" (id 4) (at 22.86 31.75 0)
-      (effects (font (size 1.27 1.27)) hide)
-    )
-    (pin "1")
-    (pin "2")
   )
   (symbol (lib_id "Device:C") (at 38.1 66.04 0) (unit 1)
@@
     (pin "1")
   )
+  (symbol (lib_id "Regulator_Switching:TSR_1-2450") (at 38.1 30.48 0) (unit 1)
+    (in_bom yes) (on_board yes) (fields_autoplaced)
+    (property "Reference" "U1" (id 0) (at 38.1 20.32 0))
+    (property "Value" "TSR_1-2450" (id 1) (at 38.1 22.86 0))
+    (property "Footprint" "Converter_DCDC:Converter_DCDC_TRACO_TSR-1_THT" (id 2) (at 38.1 34.29 0)
+      (effects (font (size 1.27 1.27) italic) (justify left) hide)
+    )
+    (property "Datasheet" "http://www.tracopower.com/products/tsr1.pdf" (id 3) (at 38.1 30.48 0)
+      (effects (font (size 1.27 1.27)) hide)
+    )
+    (pin "1")
+    (pin "2")
+    (pin "3")
+  )
   (symbol (lib_id "power:+24V") (at 22.86 27.94 0) (unit 1)
     (in_bom yes) (on_board yes) (fields_autoplaced)
@@
       (reference "#PWR02") (unit 1) (value "+24V") (footprint "")
     )
-    (path "/2151a218-87ec-4d43-b5fa-736242c52602"
-      (reference "#PWR03") (unit 1) (value "GND") (footprint "")
-    )
     (path "/86498764-3d02-46be-8f61-eaa556ccd233"
       (reference "#PWR04") (unit 1) (value "GND") (footprint "")
@@
       (reference "#PWR0104") (unit 1) (value "GND") (footprint "")
     )
-    (path "/e07c4b69-e0b4-4217-9b28-38d44f166b31"
-      (reference "C1") (unit 1) (value "10u") (footprint "Capacitor_SMD:C_1206_3216Metric")
-    )
     (path "/e4184668-3bdd-4cb2-a053-4f3d5e57b541"
       (reference "C2") (unit 1) (value "1u") (footprint "Capacitor_SMD:C_0402_1005Metric")
@@
       (reference "SW1") (unit 1) (value "SW_Push") (footprint "")
     )
-    (path "/dde4c43d-f33e-48ba-86f3-779fdfce00c2"
-      (reference "U1") (unit 1) (value "LM78M05_TO252") (footprint "Package_TO_SOT_SMD:TO-252-2")
+    (path "/fe3862ad-c819-4b65-9e75-6bbc512422a7"
+      (reference "U1") (unit 1) (value "TSR_1-2450") (footprint "Converter_DCDC:Converter_DCDC_TRACO_TSR-1_THT")
     )
     (path "/b4501435-1b74-4814-ac8d-457d48a8c57b"

Commit message: wip
Parts:
- added C1: 100n, Capacitor_SMD:C_0402_1005Metric, symbol Device:C
- added D3: CDSOT23-SM712, Octopart:Bourns_Inc.-SOT23-0-0-IPC_B, symbol Octopart:CDSOT23-SM712
- added H1, H2: MountingHole, MountingHole:MountingHole_3.5mm, symbol Mechanical:MountingHole
- added J6: 1Wire, Connector_PinHeader_2.54mm:PinHeader_1x03_P2.54mm_Vertical, symbol Connector_Generic:Conn_01x03
- added R10: 4K7, Resistor_SMD:R_0402_1005Metric, symbol Device:R_US
- J3: footprint Connector_FFC-FPC:TE_4-1734839-0_1x40-1MP_P0.5mm_Horizontal -> Connector_FFC-FPC:Hirose_FH12-40S-0.5SH_1x40-1MP_P0.50mm_Horizontal; LCSC (none) -> C506795
- R9: value R -> 330
Connections:
- net +3V3: now also C1.2, J6.2 (Pin_2), R10.1
- net GND: now also R9.2, C1.1, D3.3, J6.3 (Pin_3)
- net at D2.1 (K): now also R9.1
- net at D2.2 (A): now also U6.18 (IO15)
- net at J5.1 (Pin_1), R8.1, U2.7 (B): now also D3.1
- net at J5.2 (Pin_2), R8.2, U2.6 (A): now also D3.2
- net 1WIRE: now reaches U6.25 (IO26)
- net 1WIRE: now also J6.1 (Pin_1), R10.2
Other:
- moved on the sheet: D2, R9

Commit message: random additions
Parts:
- added C6: 10u, Capacitor_SMD:C_1206_3216Metric, symbol Device:C
- added D4: B5819W SL, Diode_SMD:D_SOD-123, symbol Device:D_Schottky
- added H3, H4: MountingHole, MountingHole:MountingHole_3.5mm, symbol Mechanical:MountingHole
- added J7: Conn_01x06, symbol Connector_Generic:Conn_01x06
- added J8: Conn_01x07, Connector_PinHeader_2.54mm:PinHeader_1x07_P2.54mm_Vertical, symbol Connector_Generic:Conn_01x07
Connections:
- net +24V: now also D4.2 (A); no longer U1.1 (Vin)
- net +3V3: now also J8.6 (Pin_6)
- net GND: now also C6.2, J8.7 (Pin_7)
- new net: C6.1, D4.1 (K), U1.1 (Vin)
- new net BLK: J8.1 (Pin_1)
- new net EXT_D/C: J8.2 (Pin_2)
- new net EXT_RESET: J8.3 (Pin_3)
- new net EXT_SCL: J8.5 (Pin_5)
- new net EXT_SDA: J8.4 (Pin_4)
Other:
- note added: "another SPI.. pinout from ST7789 board"
- moved on the sheet: C3, C4, C5, D3, H1, H2, J5, R8, U1, U2, U4
