File: UniversalControlPanel.kicad_sch (KiCad schematic)
At the start: 38 parts, among them J1 USB_B_Micro, J2 Conn_ARM_JTAG_SWD_10, J3 Conn_01x40, J4 Conn_02x03_Odd_Even, J5 Conn_01x02, J6 1Wire, J7 Conn_01x06, J8 Conn_01x07, SW1 SW_Push, U1 TSR_1-2450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

Commit message: finalizing features
Parts:
- added J9: Conn_01x02, Connector_JST:JST_XH_B2B-XH-A_1x02_P2.50mm_Vertical, symbol Connector_Generic:Conn_01x02
- added R11: 10k, Resistor_SMD:R_0402_1005Metric, symbol Device:R
- added R12: 120, Resistor_SMD:R_0805_2012Metric_Pad1.20x1.40mm_HandSolder, symbol Device:R
- added U5: SN65HVD230, Package_SO:SOIC-8_3.9x4.9mm_P1.27mm, symbol Interface_CAN_LIN:SN65HVD230
Connections:
- net EXT_D/C is gone; now on net WR(D/C): J8.2 (Pin_2)
- net EXT_RESET is gone; now on net RESET: J8.3 (Pin_3)
- net EXT_SCL is gone; now on net RS(SCL): J8.5 (Pin_5)
- net EXT_SDA is gone; now on net SDI(SDA): J8.4 (Pin_4)
- net +3V3: now also U5.3 (VCC)
- net GND: now also R11.2, U5.2 (GND)
- new net: J9.1 (Pin_1), R12.1, U5.7 (CANH)
- new net: J9.2 (Pin_2), R12.2, U5.6 (CANL)
- new net: R11.1, U5.8 (Rs)
- new net CAN0_TX: U5.1 (D)
- new net CAN_RX: U5.4 (R)
- no-connect marks 4 -> 5
Other:
- note added: "buttons and leds"

Commit message: placed
Parts:
- added J10: Conn_01x02, TerminalBlock_Phoenix:TerminalBlock_Phoenix_MKDS-1,5-2_1x02_P5.00mm_Horizontal, symbol Connector_Generic:Conn_01x02
Connections:
- net GND: now also J10.2 (Pin_2)
- net +24V renamed 24V
- net 24V: now also J10.1 (Pin_1)
Other:
- moved on the sheet: C3, C4, C5, C6, D4, U1, U4

Commit message: added switch
Parts:
- added J11: Conn_01x02, Connector_JST:JST_XH_B2B-XH-A_1x02_P2.50mm_Vertical, symbol Connector_Generic:Conn_01x02
- added JP1, JP2: Jumper_2_Bridged, Jumper:SolderJumper-2_P1.3mm_Bridged2Bar_Pad1.0x1.5mm, symbol Jumper:Jumper_2_Bridged
- SW1: footprint (none) -> Local:TS-1187A-B-A-B
Connections:
- net CAN_RX: now also JP2.1 (A); no longer U5.4 (R)
- net CAN0_TX: no longer names the net of U5.1 (D)
- net CAN0_TX: now also J11.1 (Pin_1), JP1.2 (B)
- new net: J11.2 (Pin_2), JP2.2 (B), U5.4 (R)
- new net CAN_TX: JP1.1 (A)
Changed lines of the file:
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@@
   (junction (at 254 152.4) (diameter 0) (color 0 0 0 0)
   )
+  (junction (at 145.796 132.08) (diameter 0) (color 0 0 0 0)
+  )
   (junction (at 46.99 168.91) (diameter 0) (color 0 0 0 0)
   )
@@
   )
   (junction (at 22.86 106.68) (diameter 0) (color 0 0 0 0)
+  )
+  (junction (at 144.018 129.54) (diameter 0) (color 0 0 0 0)
   )
   (junction (at 254 119.38) (diameter 0) (color 0 0 0 0)
@@
     (stroke (width 0) (type default) (color 0 0 0 0))
   )
+  (wire (pts (xy 145.796 132.08) (xy 152.4 132.08))
+    (stroke (width 0) (type default) (color 0 0 0 0))
+  )
   (wire (pts (xy 74.93 27.94) (xy 81.28 27.94))
     (stroke (width 0) (type default) (color 0 0 0 0))
@@
     (stroke (width 0) (type default) (color 0 0 0 0))
   )
+  (wire (pts (xy 143.51 132.08) (xy 145.796 132.08))
+    (stroke (width 0) (type default) (color 0 0 0 0))
+  )
   (wire (pts (xy 254 116.84) (xy 254 119.38))
     (stroke (width 0) (type default) (color 0 0 0 0))
@@
     (stroke (width 0) (type default) (color 0 0 0 0))
   )
+  (wire (pts (xy 111.76 144.018) (xy 118.618 144.018))
+    (stroke (width 0) (type default) (color 0 0 0 0))
+  )
   (wire (pts (xy 20.32 104.14) (xy 20.32 106.68))
     (stroke (width 0) (type default) (color 0 0 0 0))
@@
     (stroke (width 0) (type default) (color 0 0 0 0))
   )
+  (wire (pts (xy 111.252 134.874) (xy 118.364 134.874))
+    (stroke (width 0) (type default) (color 0 0 0 0))
+  )
   (wire (pts (xy 179.07 129.54) (xy 186.69 129.54))
     (stroke (width 0) (type default) (color 0 0 0 0))
@@
     (stroke (width 0) (type default) (color 0 0 0 0))
   )
+  (wire (pts (xy 144.018 129.54) (xy 152.4 129.54))
+    (stroke (width 0) (type default) (color 0 0 0 0))
+  )
   (wire (pts (xy 33.02 59.69) (xy 38.1 59.69))
     (stroke (width 0) (type default) (color 0 0 0 0))
@@
     (stroke (width 0) (type default) (color 0 0 0 0))
   )
+  (wire (pts (xy 145.796 144.018) (xy 145.796 132.08))
+    (stroke (width 0) (type default) (color 0 0 0 0))
+  )
   (wire (pts (xy 254 88.9) (xy 254 91.44))
     (stroke (width 0) (type default) (color 0 0 0 0))
@@
     (stroke (width 0) (type default) (color 0 0 0 0))
   )
+  (wire (pts (xy 128.778 144.018) (xy 145.796 144.018))
+    (stroke (width 0) (type default) (color 0 0 0 0))
+  )
   (wire (pts (xy 242.57 83.82) (xy 257.81 83.82))
     (stroke (width 0) (type default) (color 0 0 0 0))
@@
     (stroke (width 0) (type default) (color 0 0 0 0))
   )
-  (wire (pts (xy 143.51 132.08) (xy 152.4 132.08))
-    (stroke (width 0) (type default) (color 0 0 0 0))
-  )
   (wire (pts (xy 144.78 177.8) (xy 144.78 179.07))
     (stroke (width 0) (type default) (color 0 0 0 0))
@@
     (stroke (width 0) (type default) (color 0 0 0 0))
   )
-  (wire (pts (xy 143.51 129.54) (xy 152.4 129.54))
+  (wire (pts (xy 143.51 129.54) (xy 144.018 129.54))
     (stroke (width 0) (type default) (color 0 0 0 0))
   )
@@
     (stroke (width 0) (type default) (color 0 0 0 0))
   )
+  (wire (pts (xy 144.018 134.874) (xy 128.524 134.874))
+    (stroke (width 0) (type default) (color 0 0 0 0))
+  )
   (wire (pts (xy 254 121.92) (xy 257.81 121.92))
     (stroke (width 0) (type default) (color 0 0 0 0))
@@
   )
   (wire (pts (xy 146.05 49.53) (xy 146.05 58.42))
+    (stroke (width 0) (type default) (color 0 0 0 0))
+  )
+  (wire (pts (xy 144.018 129.54) (xy 144.018 134.874))
     (stroke (width 0) (type default) (color 0 0 0 0))
   )
@@
     (effects (font (size 1.27 1.27)) (justify left bottom))
   )
-  (label "CAN_RX" (at 143.51 132.08 0)
+  (label "CAN_RX" (at 111.76 144.018 0)
     (effects (font (size 1.27 1.27)) (justify left bottom))
   )
@@
     (effects (font (size 1.27 1.27)) (justify left bottom))
   )
-  (label "CAN0_TX" (at 143.51 129.54 0)
-    (effects (font (size 1.27 1.27)) (justify left bottom))
-  )
   (label "RESET" (at 242.57 68.58 0)
     (effects (font (size 1.27 1.27)) (justify left bottom))
@@
   )
   (label "TMS" (at 229.87 35.56 0)
+    (effects (font (size 1.27 1.27)) (justify left bottom))
+  )
+  (label "CAN_TX" (at 111.252 134.874 0)
     (effects (font (size 1.27 1.27)) (justify left bottom))
   )
@@
     (property "Reference" "SW1" (id 0) (at 27.94 52.07 0))
     (property "Value" "SW_Push" (id 1) (at 27.94 54.61 0))
-    (property "Footprint" "" (id 2) (at 27.94 54.61 0)
+    (property "Footprint" "Local:TS-1187A-B-A-B" (id 2) (at 27.94 54.61 0)
       (effects (font (size 1.27 1.27)) hide)
     )
@@
     )
   )
+  (symbol (lib_id "Jumper:Jumper_2_Bridged") (at 123.698 144.018 0) (unit 1)
+    (in_bom yes) (on_board yes) (fields_autoplaced)
+    (property "Reference" "JP2" (id 0) (at 123.698 137.668 0))
+    (property "Value" "Jumper_2_Bridged" (id 1) (at 123.698 140.208 0))
+    (property "Footprint" "Jumper:SolderJumper-2_P1.3mm_Bridged2Bar_Pad1.0x1.5mm" (id 2) (at 123.698 144.018 0)
+      (effects (font (size 1.27 1.27)) hide)
+    )
+    (property "Datasheet" "~" (id 3) (at 123.698 144.018 0)
+      (effects (font (size 1.27 1.27)) hide)
+    )
+    (pin "1")
+    (pin "2")
+  )
   (symbol (lib_id "Connector_Generic:Conn_01x07") (at 226.06 109.22 0) (unit 1)
     (in_bom yes) (on_board yes) (fields_autoplaced)
@@
     )
     (pin "1")
+  )
+  (symbol (lib_id "Connector_Generic:Conn_01x02") (at 138.43 129.54 0) (mirror y) (unit 1)
+    (in_bom yes) (on_board yes) (fields_autoplaced)
+    (property "Reference" "J11" (id 0) (at 138.43 122.936 0))
+    (property "Value" "Conn_01x02" (id 1) (at 138.43 125.476 0))
+    (property "Footprint" "Connector_JST:JST_XH_B2B-XH-A_1x02_P2.50mm_Vertical" (id 2) (at 138.43 129.54 0)
+      (effects (font (size 1.27 1.27)) hide)
+    )
+    (property "Datasheet" "~" (id 3) (at 138.43 129.54 0)
+      (effects (font (size 1.27 1.27)) hide)
+    )
+    (pin "1")
+    (pin "2")
   )
   (symbol (lib_id "power:GND") (at 124.46 181.61 0) (unit 1)
@@
     )
     (property "Datasheet" "~" (id 3) (at 38.1 66.04 0)
+      (effects (font (size 1.27 1.27)) hide)
+    )
+    (pin "1")
+    (pin "2")
+  )
+  (symbol (lib_id "Jumper:Jumper_2_Bridged") (at 123.444 134.874 0) (unit 1)
+    (in_bom yes) (on_board yes) (fields_autoplaced)
+    (property "Reference" "JP1" (id 0) (at 123.444 128.524 0))
+    (property "Value" "Jumper_2_Bridged" (id 1) (at 123.444 131.064 0))
+    (property "Footprint" "Jumper:SolderJumper-2_P1.3mm_Bridged2Bar_Pad1.0x1.5mm" (id 2) (at 123.444 134.874 0)
+      (effects (font (size 1.27 1.27)) hide)
+    )
+    (property "Datasheet" "~" (id 3) (at 123.444 134.874 0)
       (effects (font (size 1.27 1.27)) hide)
     )
@@
       (reference "J10") (unit 1) (value "Conn_01x02") (footprint "TerminalBlock_Phoenix:TerminalBlock_Phoenix_MKDS-1,5-2_1x02_P5.00mm_Horizontal")
     )
+    (path "/a20106a5-7c6c-476e-9e8e-7784d2dfd43d"
+      (reference "J11") (unit 1) (value "Conn_01x02") (footprint "Connector_JST:JST_XH_B2B-XH-A_1x02_P2.50mm_Vertical")
+    )
+    (path "/e6f55e57-c10f-46cf-985f-7a37dbbf9653"
+      (reference "JP1") (unit 1) (value "Jumper_2_Bridged") (footprint "Jumper:SolderJumper-2_P1.3mm_Bridged2Bar_Pad1.0x1.5mm")
+    )
+    (path "/906d436e-f9a5-4903-b1fb-3eb672bf2619"
+      (reference "JP2") (unit 1) (value "Jumper_2_Bridged") (footprint "Jumper:SolderJumper-2_P1.3mm_Bridged2Bar_Pad1.0x1.5mm")
+    )
     (path "/f220d6a7-3170-4e04-8de6-2df0c3962fe0"
       (reference "R1") (unit 1) (value "10k") (footprint "Resistor_SMD:R_0402_1005Metric")
@@
     )
     (path "/0e592cd4-1950-44ef-9727-8e526f4c4e12"
-      (reference "SW1") (unit 1) (value "SW_Push") (footprint "")
+      (reference "SW1") (unit 1) (value "SW_Push") (footprint "Local:TS-1187A-B-A-B")
     )
     (path "/fe3862ad-c819-4b65-9e75-6bbc512422a7"

Commit message: restart work
Parts:
- removed D1: B5819W SL, Diode_SMD:D_SOD-123, symbol Device:D_Schottky
- removed D3: CDSOT23-SM712, Octopart:Bourns_Inc.-SOT23-0-0-IPC_B, symbol Octopart:CDSOT23-SM712
- removed J1: USB_B_Micro, Connector_USB:USB_Mini-B_Tensility_54-00023_Vertical, symbol Connector:USB_B_Micro
- removed J2: Conn_ARM_JTAG_SWD_10, Connector_PinHeader_1.27mm:PinHeader_2x05_P1.27mm_Vertical, symbol Connector:Conn_ARM_JTAG_SWD_10
- removed J6: 1Wire, Connector_PinHeader_2.54mm:PinHeader_1x03_P2.54mm_Vertical, symbol Connector_Generic:Conn_01x03
- removed J7: Conn_01x06, symbol Connector_Generic:Conn_01x06
- removed R10: 4K7, Resistor_SMD:R_0402_1005Metric, symbol Device:R_US
- removed U3: USBLC6-2SC6, Package_TO_SOT_SMD:SOT-23-6, symbol Power_Protection:USBLC6-2SC6
- added BTNS1: Conn_01x06, Connector_JST:JST_XH_B6B-XH-A_1x06_P2.50mm_Vertical, symbol Connector_Generic:Conn_01x06
- added C7, C8, C9: 100n/16V, Capacitor_SMD:C_0402_1005Metric, symbol Device:C
- added D3: LED_BLUE, LED_SMD:LED_0603_1608Metric, symbol Device:LED
- added D5: LED_GREEN, LED_SMD:LED_0603_1608Metric, symbol Device:LED
- added F1: 2920L050DR, Fuse:Fuse_2920_7451Metric, symbol Device:Polyfuse
- added IC1: PSM712-LF-T7, Package_TO_SOT_SMD:SOT-23, symbol _Local:PSM712-LF-T7
- added Q1, Q2: 2N7002, Package_TO_SOT_SMD:SOT-23, symbol Transistor_FET:2N7002
- added R13, R14: 22, Resistor_SMD:R_0402_1005Metric, symbol Device:R
- added R15, R16: 100k, Resistor_SMD:R_0402_1005Metric, symbol Device:R
- added R17, R18: 5k6, Resistor_SMD:R_0402_1005Metric, symbol Device:R
- added R19, R20: 75k, Resistor_SMD:R_0402_1005Metric, symbol Device:R
- C1: now left out of the parts list
Connections:
- net +3V3: now also BTNS1.5 (Pin_5), C9.1, R19.1, R20.1; no longer C1.2
- net 24V: now also F1.1; no longer D4.2 (A)
- net GND: now also D4.2 (A), BTNS1.6 (Pin_6), C7.2, C8.2, C9.2, D3.1 (K), D5.1 (K), IC1.3 (GND), Q1.2 (S), Q2.2 (S), R15.2, R16.2
- net at J5.1 (Pin_1), R8.1, U2.7 (B): now also IC1.1 (I/O_1)
- net at J5.2 (Pin_2), R8.2, U2.6 (A): now also IC1.2 (I/O_2)
- net at C6.1, D4.1 (K), U1.1 (Vin): now also F1.2
- new net: BTNS1.2 (Pin_2), R18.2, R19.2
- new net: BTNS1.1 (Pin_1), C1.2, R17.2, R20.2
- new net: D5.2 (A), R14.1
- new net: BTNS1.4 (Pin_4), Q2.3 (D)
- new net: BTNS1.3 (Pin_3), Q1.3 (D)
- new net: D3.2 (A), R13.1
- new net BTN1: C7.1, R17.1
- new net BTN2: C8.1, R18.1
- new net LED1: Q1.1 (G), R14.2, R15.1
- new net LED2: Q2.1 (G), R13.2, R16.1
- no-connect marks 5 -> 4
Other:
- note added: "if 1WIRE is needed, replace R20 with 4k7 and populate C1"
- note removed: "buttons and leds"
- note removed: "perhaps a R (22E) and C to GND (22p)"
- moved on the sheet: C2, C3, C4, C5, C6, D4, R1, SW1, U1, U4

Commit message: wired
Parts:
- removed C3: 10u, Capacitor_SMD:C_1206_3216Metric, symbol Device:C
- removed D2: LED, LED_SMD:LED_0603_1608Metric, symbol Device:LED
- removed J11: Conn_01x02, Connector_JST:JST_XH_B2B-XH-A_1x02_P2.50mm_Vertical, symbol Connector_Generic:Conn_01x02
- removed JP2: Jumper_2_Bridged, Jumper:SolderJumper-2_P1.3mm_Bridged2Bar_Pad1.0x1.5mm, symbol Jumper:Jumper_2_Bridged
- removed R9: 330, Resistor_SMD:R_0402_1005Metric, symbol Device:R
- removed U4: AMS1117-3.3, Package_TO_SOT_SMD:SOT-223-3_TabPin2, symbol Regulator_Linear:AMS1117-3.3
- added JP2, JP4: Jumper_3_Bridged12, Jumper:SolderJumper-3_P1.3mm_Bridged2Bar12_RoundedPad1.0x1.5mm, symbol Jumper:Jumper_3_Bridged12
- added JP3: Jumper_2_Bridged, Jumper:SolderJumper-2_P1.3mm_Bridged2Bar_RoundedPad1.0x1.5mm, symbol Jumper:Jumper_2_Bridged
- J10: footprint TerminalBlock_Phoenix:TerminalBlock_Phoenix_MKDS-1,5-2_1x02_P5.00mm_Horizontal -> _Local:1985807
- JP1: footprint Jumper:SolderJumper-2_P1.3mm_Bridged2Bar_Pad1.0x1.5mm -> Jumper:SolderJumper-2_P1.3mm_Bridged2Bar_RoundedPad1.0x1.5mm
- U1: value TSR_1-2450 -> TSR_1-2433
Connections:
- net BTN1 is gone; now on net TDI: C7.1, R17.1
- net BTN2 is gone; now on net TMS: C8.1, R18.1
- net LED1 is gone; now on net TDO: Q1.1 (G), R14.2, R15.1
- net LED2 is gone; now on net TCK: Q2.1 (G), R13.2, R16.1
- net +3V3: now also U1.3 (Vout)
- net +5V: no longer U1.3 (Vout)
- net U1RXD: now also JP4.2 (C); no longer U2.1 (RO)
- net U1TXD: now also JP2.2 (C); no longer U2.4 (DI)
- net at U6.18 (IO15): now also JP3.2 (B)
- net at JP1.2 (B): now also U6.17 (IO14); no longer U5.1 (D)
- net R(CRX): now reaches U5.4 (R)
- net R(CRX): now also JP4.1 (A)
- net CAN_TX renamed DI
- net DI: now also U2.4 (DI), JP2.3 (B)
- new net D(CTX): JP2.1 (A), U5.1 (D)
- new net RO: JP3.1 (A), JP4.3 (B), U2.1 (RO)
Other:
- moved on the sheet: C4, C5, C9, IC1, J5, J9, R11, R12, R8, U2, U5

Commit message: before reversing display
Parts:
- removed BTNS1: Conn_01x06, Connector_JST:JST_XH_B6B-XH-A_1x06_P2.50mm_Vertical, symbol Connector_Generic:Conn_01x06
- removed J5: Conn_01x02, Connector_JST:JST_XH_B2B-XH-A_1x02_P2.50mm_Vertical, symbol Connector_Generic:Conn_01x02
- removed J8: Conn_01x07, Connector_PinHeader_2.54mm:PinHeader_1x07_P2.54mm_Vertical, symbol Connector_Generic:Conn_01x07
- added C10, C11, C3: 100n/16V, Capacitor_SMD:C_0402_1005Metric, symbol Device:C
- added J1: Conn_01x09, Connector_JST:JST_XH_B9B-XH-A_1x09_P2.50mm_Vertical, symbol Connector_Generic:Conn_01x09
- added J2: Conn_01x09, Connector_PinHeader_2.54mm:PinHeader_1x09_P2.54mm_Vertical, symbol Connector_Generic:Conn_01x09
- added J5: Conn_01x03, Connector_JST:JST_XH_B3B-XH-A_1x03_P2.50mm_Vertical, symbol Connector_Generic:Conn_01x03
- added J6: Conn_01x07, Connector_PinHeader_2.54mm:PinHeader_1x07_P2.54mm_Vertical, symbol Connector_Generic:Conn_01x07
- added Q3: 2N7002, Package_TO_SOT_SMD:SOT-23, symbol Transistor_FET:2N7002
- added R10, R22: 15k, Resistor_SMD:R_0402_1005Metric, symbol Device:R
- added R21, R9: 8k2, Resistor_SMD:R_0402_1005Metric, symbol Device:R
- added U3: L78L05_SOT89, Package_TO_SOT_SMD:SOT-89-3, symbol Regulator_Linear:L78L05_SOT89
- C4: value 100n -> 100n/16V
- R4, R5, R6, R7: value R -> 68R
Connections:
- net +3V3: now also C10.1, C3.1, J1.5 (Pin_5), J2.9 (Pin_9), J6.6 (Pin_6)
- net +5V: now also C11.1, J1.8 (Pin_8), U3.1 (OUT)
- net 24V: now also C6.1, D4.1 (K), F1.2, U1.1 (Vin), U3.3 (IN); no longer F1.1, J10.1 (Pin_1)
- net BLK: now also U6.16 (IO13), J2.8 (Pin_8), J6.1 (Pin_1)
- net GND: now also C10.2, C11.2, C3.2, J1.9 (Pin_9), J2.2 (Pin_2), J5.3 (Pin_3), J6.7 (Pin_7), Q3.2 (S), R10.2, R22.2, U3.2 (GND); no longer R4.1, R5.2, R6.1, R7.2
- net RESET: now also J2.7 (Pin_7), J6.3 (Pin_3)
- net RS(SCL): now also J2.5 (Pin_5), J6.5 (Pin_5)
- net SDI(SDA): now also J2.4 (Pin_4), J6.4 (Pin_4)
- net SDO: now also J2.6 (Pin_6)
- net WR(D/C): now also J2.3 (Pin_3), J6.2 (Pin_2)
- net at IC1.1 (I/O_1), R8.1, U2.7 (B): now also J5.1 (Pin_1)
- net at IC1.2 (I/O_2), R8.2, U2.6 (A): now also J5.2 (Pin_2)
- net at R18.2, R19.2: now also J1.2 (Pin_2)
- net at C1.2, R17.2, R20.2: now also J1.1 (Pin_1)
- net at U6.14 (IO11): now also R10.1, R9.2
- net at U6.15 (IO12): now also R21.2, R22.1
- net at U6.24 (IO21): now also Q3.1 (G)
- net at Q2.3 (D): now also J1.4 (Pin_4)
- net at Q1.3 (D): now also J1.3 (Pin_3)
- net 1WIRE renamed CS2
- net CS2: now also J2.1 (Pin_1)
- new net: Q3.3 (D), R4.1, R5.2, R6.1, R7.2
- new net: J1.6 (Pin_6), R9.1
- new net: J1.7 (Pin_7), R21.1
- new net IN_PWR: F1.1, J10.1 (Pin_1)
Other:
- moved on the sheet: C9

Commit message: before upload
Parts:
- removed JP2, JP4: Jumper_3_Bridged12, Jumper:SolderJumper-3_P1.3mm_Bridged2Bar12_RoundedPad1.0x1.5mm, symbol Jumper:Jumper_3_Bridged12
- added JP2, JP4: Jumper_2_Bridged, Jumper:SolderJumper-2_P1.3mm_Bridged2Bar_RoundedPad1.0x1.5mm, symbol Jumper:Jumper_2_Bridged
- D4: LCSC (none) -> C8598
- F1: now left out of the parts list
- R1, R11, R2, R3: LCSC (none) -> C25744
- R4, R5, R6, R7: value 68R -> 75; LCSC (none) -> C25133
- SW1: LCSC (none) -> C318884
- U2: LCSC (none) -> C559550
- U6: LCSC (none) -> C967026
Connections:
- net +3V3: now also J3.29 (Pin_29), J3.38 (Pin_38); no longer J3.12 (Pin_12), J3.3 (Pin_3)
- net +5V: now also J3.8 (Pin_8); no longer J3.33 (Pin_33)
- net BLK: now also Q3.1 (G), U6.4 (IO01); no longer J2.8 (Pin_8), U6.16 (IO13)
- net CS: now also J3.32 (Pin_32); no longer J3.9 (Pin_9)
- net CTP-INT: now also J3.36 (Pin_36); no longer J3.5 (Pin_5)
- net CTP-RST: now also J3.10 (Pin_10); no longer J3.31 (Pin_31)
- net CTP-SCL: now also J3.35 (Pin_35); no longer J3.6 (Pin_6)
- net CTP-SDA: now also J3.9 (Pin_9); no longer J3.32 (Pin_32)
- net D(CTX): now also JP2.1 (A)
- net GND: now also J3.11 (Pin_11), J3.12 (Pin_12), J3.13 (Pin_13); no longer J3.28 (Pin_28), J3.29 (Pin_29), J3.30 (Pin_30)
- net LEDK1: now also J3.7 (Pin_7); no longer J3.34 (Pin_34)
- net LEDK2: now also J3.6 (Pin_6); no longer J3.35 (Pin_35)
- net LEDK3: now also J3.5 (Pin_5); no longer J3.36 (Pin_36)
- net LEDK4: now also J3.4 (Pin_4); no longer J3.37 (Pin_37)
- net R(CRX): now also JP4.1 (A)
- net RESET: now also J3.34 (Pin_34); no longer J3.7 (Pin_7)
- net RS(SCL): now also J3.33 (Pin_33); no longer J3.8 (Pin_8)
- net SDI(SDA): now also J3.39 (Pin_39); no longer J3.2 (Pin_2)
- net SDO: now also J3.28 (Pin_28); no longer J3.13 (Pin_13)
- net U1RXD: now also JP4.2 (B)
- net U1TXD: now also JP2.2 (B)
- net WR(D/C): now also J3.30 (Pin_30); no longer J3.11 (Pin_11)
- net at U6.24 (IO21): no longer Q3.1 (G)
- new net RND: J2.8 (Pin_8), U6.16 (IO13)
Other:
- note added: "Warning: this is reversed pinout to match connector"
