File: UniversalControlPanel.kicad_pcb (KiCad board)
At the start: 2 copper layers, 65 x 55 mm, 31 parts, among them J1 USB_B_Micro, J2 Conn_ARM_JTAG_SWD_10, J3 Conn_01x40, J4 Conn_02x03_Odd_Even, J5 Conn_01x02, J6 1Wire, U1 TSR_1-2450, U2 MAX14783ExS, U3 USBLC6-2SC6, U4 AMS1117-3.3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

Commit message: random additions
Parts:
- added C6: 10u, Capacitor_SMD:C_1206_3216Metric, F.Cu at (140.0, 129.0)
- added D4: B5819W SL, Diode_SMD:D_SOD-123, F.Cu at (134.3, 129.0)
- added H3: MountingHole, MountingHole:MountingHole_3.5mm, F.Cu at (168.0, 81.0)
- added H4: MountingHole, MountingHole:MountingHole_3.5mm, F.Cu at (168.0, 130.0)
- added J8: Conn_01x07, Connector_PinHeader_2.54mm:PinHeader_1x07_P2.54mm_Vertical, F.Cu at (124.0, 98.0)
- moved D2 15.3 mm to (157.0, 89.0)
- moved R9 12.5 mm to (160.0, 91.5)
- moved J2 3.71 mm to (157.0, 130.0)
- moved U1 1.68 mm to (150.0, 126.4)
Connections:
- U1 pad 1: +24V -> Net-(U1-Pad1)

Commit message: finalizing features
Parts:
- added J9: Conn_01x02, Connector_JST:JST_XH_B2B-XH-A_1x02_P2.50mm_Vertical, F.Cu at (137.0, 139.0)
- added R11: 10k, Resistor_SMD:R_0402_1005Metric, F.Cu at (144.4, 143.1)
- added R12: 120, Resistor_SMD:R_0805_2012Metric_Pad1.20x1.40mm_HandSolder, F.Cu at (135.9, 144.9)
- added U5: SN65HVD230, Package_SO:SOIC-8_3.9x4.9mm_P1.27mm, F.Cu at (147.2, 138.8)

Commit message: connector finalized
Parts:
- moved J1 28.1 mm to (141.8, 97.2), turned to 0 degrees
- moved U3 24.0 mm to (142.8, 104.0)
- moved R12 21.3 mm to (138.6, 123.8)
- moved D4 17.4 mm to (149.6, 120.7)
- moved C6 14.8 mm to (149.4, 117.6)
- moved R11 11.1 mm to (141.8, 132.3)
- moved U5 11.1 mm to (144.6, 128.1)
- moved J9 10.0 mm to (136.5, 129.0), turned to 180 degrees
- moved J2 9.72 mm to (155.0, 120.5)
- moved U1 4.93 mm to (153.6, 129.8), turned to 0 degrees
- moved J3 4.61 mm to (118.2, 104.4)
- moved U6 4.50 mm to (163.0, 105.5)
- moved H3 4.01 mm to (172.0, 81.2)
- moved H4 4.01 mm to (172.0, 129.8)
Connections:
- J8 pad 2: /EXT_D/C -> /WR(D/C)
- J8 pad 3: /EXT_RESET -> /RESET
- J8 pad 4: /EXT_SDA -> /SDI(SDA)
- J8 pad 5: /EXT_SCL -> /RS(SCL)
Other:
- board size 65 x 55 mm -> 70 x 55 mm

Commit message: placed
Parts:
- added J10: Conn_01x02, TerminalBlock_Phoenix:TerminalBlock_Phoenix_MKDS-1,5-2_1x02_P5.00mm_Horizontal, F.Cu at (129.6, 83.8)
- J1: moved to F.Cu
- J8: moved to B.Cu
- moved J5 59.6 mm to (162.7, 81.2), turned to 0 degrees
- moved C2 51.8 mm to (175.0, 122.0)
- moved U2 50.7 mm to (171.1, 89.0), turned to 180 degrees
- moved D3 50.5 mm to (164.0, 89.6), turned to 180 degrees
- moved R8 50.2 mm to (164.0, 86.4), turned to 0 degrees
- moved R1 43.2 mm to (172.7, 122.0)
- moved R6 39.9 mm to (122.5, 114.2), turned to 180 degrees
- moved C4 38.7 mm to (174.7, 99.5)
- moved U1 38.2 mm to (131.7, 98.5), turned to -90 degrees
- moved D4 35.8 mm to (129.7, 90.9), turned to 180 degrees
- moved R7 33.5 mm to (122.5, 115.7)
- moved R4 32.0 mm to (122.5, 111.4), turned to 180 degrees
- moved R5 31.6 mm to (122.5, 112.9)
- moved C6 31.3 mm to (127.6, 95.2), turned to -90 degrees
- moved C3 28.9 mm to (127.7, 100.8), turned to 90 degrees
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Connections:
- D4 pad 2: +24V -> /24V

Commit message: movin st7789
Parts:
- moved J8 6.01 mm to (135.8, 97.5)
- moved C3 4.22 mm to (123.5, 100.8)
- moved C6 4.22 mm to (123.4, 95.1)
- moved C1 4.22 mm to (124.5, 104.7)
- moved U1 4.22 mm to (127.5, 98.5)
Changed lines of the file:
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@@
   )
   (footprint "Capacitor_SMD:C_1206_3216Metric" (layer "F.Cu")
-    (at 127.6 95.15 -90)
+    (at 123.3825 95.0575 -90)
     (descr "Capacitor SMD 1206 (3216 Metric), square (rectangular) end terminal, IPC_7351 nominal, (Body size source: IPC-SM-782 page 76, https://www.pcb-3d.com/wordpress/wp-content/uploads/ipc-sm-782a_amendment_1_and_2.pdf), generated with kicad-footprint-generator")
     (tags "capacitor")
@@
   )
   (footprint "Converter_DCDC:Converter_DCDC_TRACO_TSR-1_THT" (layer "F.Cu")
-    (at 131.6675 98.5425 -90)
+    (at 127.45 98.45 -90)
     (descr "DCDC-Converter, TRACO, TSR 1-xxxx")
     (tags "DCDC-Converter TRACO TSR-1")
@@
   )
   (footprint "Capacitor_SMD:C_1206_3216Metric" (layer "F.Cu")
-    (at 127.675 100.85 90)
+    (at 123.4575 100.7575 90)
     (descr "Capacitor SMD 1206 (3216 Metric), square (rectangular) end terminal, IPC_7351 nominal, (Body size source: IPC-SM-782 page 76, https://www.pcb-3d.com/wordpress/wp-content/uploads/ipc-sm-782a_amendment_1_and_2.pdf), generated with kicad-footprint-generator")
     (tags "capacitor")
@@
   )
   (footprint "Capacitor_SMD:C_0402_1005Metric" (layer "F.Cu")
-    (at 128.7 104.8 -90)
+    (at 124.4825 104.7075 -90)
     (descr "Capacitor SMD 0402 (1005 Metric), square (rectangular) end terminal, IPC_7351 nominal, (Body size source: IPC-SM-782 page 76, https://www.pcb-3d.com/wordpress/wp-content/uploads/ipc-sm-782a_amendment_1_and_2.pdf), generated with kicad-footprint-generator")
     (tags "capacitor")
@@
   )
   (footprint "Connector_PinHeader_2.54mm:PinHeader_1x07_P2.54mm_Vertical" (layer "B.Cu")
-    (at 141.7 96.65 180)
+    (at 135.75 97.525 180)
     (descr "Through hole straight pin header, 1x07, 2.54mm pitch, single row")
     (tags "Through hole pin header THT 1x07 2.54mm single row")
@@
   )
   (gr_line (start 121 114.6) (end 120.9 94.1) (layer "Dwgs.User") (width 0.15))
+  (gr_rect (start 133.25 92.425) (end 162.55 118.625) (layer "Dwgs.User") (width 0.15) (fill none))
+  (gr_line (start 113.025 133) (end 183 78) (layer "Dwgs.User") (width 0.15))
+  (gr_line (start 113 78) (end 183 133) (layer "Dwgs.User") (width 0.15))
   (gr_line (start 121 114.6) (end 113 114.6) (layer "Dwgs.User") (width 0.15))
   (gr_line (start 120.9 94.1) (end 113 94.1) (layer "Dwgs.User") (width 0.15))

Commit message: added switch
Parts:
- added J11: Conn_01x02, Connector_JST:JST_XH_B2B-XH-A_1x02_P2.50mm_Vertical, F.Cu at (126.7, 128.7)
- added JP1: Jumper_2_Bridged, Jumper:SolderJumper-2_P1.3mm_Bridged2Bar_Pad1.0x1.5mm, F.Cu at (127.8, 122.5)
- added JP2: Jumper_2_Bridged, Jumper:SolderJumper-2_P1.3mm_Bridged2Bar_Pad1.0x1.5mm, F.Cu at (124.2, 122.5)
- added SW1: SW_Push, Local:TS-1187A-B-A-B, F.Cu at (145.2, 128.4)
- moved R11 12.0 mm to (144.0, 111.2)
- moved R12 11.6 mm to (134.0, 124.0)
- moved J9 9.89 mm to (135.5, 128.7)
- moved U5 6.24 mm to (134.4, 119.0)
Connections:
- U5 pad 1: /CAN0_TX -> Net-(U5-Pad1)
- U5 pad 4: /CAN_RX -> Net-(U5-Pad4)

Commit message: restart work
Parts:
- removed D1: B5819W SL, Diode_SMD:D_SOD-123
- removed J1: USB_B_Micro, Connector_USB:USB_Mini-B_Tensility_54-00023_Vertical
- removed J2: Conn_ARM_JTAG_SWD_10, Connector_PinHeader_1.27mm:PinHeader_2x05_P1.27mm_Vertical
- removed J6: 1Wire, Connector_PinHeader_2.54mm:PinHeader_1x03_P2.54mm_Vertical
- removed R10: 4K7, Resistor_SMD:R_0402_1005Metric
- removed U3: USBLC6-2SC6, Package_TO_SOT_SMD:SOT-23-6
- added BTNS1: Conn_01x06, Connector_JST:JST_XH_B6B-XH-A_1x06_P2.50mm_Vertical, F.Cu at (145.0, 139.0)
- added C7: 100n/16V, Capacitor_SMD:C_0402_1005Metric, F.Cu at (167.3, 140.6)
- added C8: 100n/16V, Capacitor_SMD:C_0402_1005Metric, F.Cu at (167.3, 138.6)
- added C9: 100n/16V, Capacitor_SMD:C_0402_1005Metric, F.Cu at (155.7, 149.0)
- added D5: LED_GREEN, LED_SMD:LED_0603_1608Metric, F.Cu at (143.6, 149.2)
- added IC1: PSM712-LF-T7, Package_TO_SOT_SMD:SOT-23, F.Cu at (163.4, 137.8)
- added Q1: 2N7002, Package_TO_SOT_SMD:SOT-23, F.Cu at (163.4, 142.3)
- added Q2: 2N7002, Package_TO_SOT_SMD:SOT-23, F.Cu at (149.1, 145.7)
- added R13: 22, Resistor_SMD:R_0402_1005Metric, F.Cu at (152.8, 149.0)
- added R14: 22, Resistor_SMD:R_0402_1005Metric, F.Cu at (153.0, 147.0)
- added R15: 100k, Resistor_SMD:R_0402_1005Metric, F.Cu at (160.0, 145.5)
- added R16: 100k, Resistor_SMD:R_0402_1005Metric, F.Cu at (167.3, 136.6)
- added R17: 5k6, Resistor_SMD:R_0402_1005Metric, F.Cu at (149.9, 148.9)
- added R18: 5k6, Resistor_SMD:R_0402_1005Metric, F.Cu at (157.1, 144.4)
- added R19: 75k, Resistor_SMD:R_0402_1005Metric, F.Cu at (147.0, 148.9)
- added R20: 75k, Resistor_SMD:R_0402_1005Metric, F.Cu at (155.9, 147.0)
- D3: value CDSOT23-SM712 -> LED_BLUE; footprint Octopart:Bourns_Inc.-SOT23-0-0-IPC_B -> LED_SMD:LED_0603_1608Metric
- moved D3 56.1 mm to (153.6, 144.7), turned to 0 degrees
- moved C1 38.8 mm to (125.0, 143.5), turned to 0 degrees
Connections:
- C1 pad 2: +3V3 -> Net-(BTNS1-Pad1)
- D3 pad 1: Net-(D3-Pad1) -> GND
- D4 pad 2: /24V -> GND
- J5 pad 1: Net-(D3-Pad1) -> Net-(J5-Pad1)
- J5 pad 2: Net-(D3-Pad2) -> Net-(J5-Pad2)
- R8 pad 1: Net-(D3-Pad1) -> Net-(J5-Pad1)
- R8 pad 2: Net-(D3-Pad2) -> Net-(J5-Pad2)
- U2 pad 6: Net-(D3-Pad2) -> Net-(J5-Pad2)
- U2 pad 7: Net-(D3-Pad1) -> Net-(J5-Pad1)

Commit message: wired
Parts:
- removed C3: 10u, Capacitor_SMD:C_1206_3216Metric
- removed D2: LED, LED_SMD:LED_0603_1608Metric
- removed J11: Conn_01x02, Connector_JST:JST_XH_B2B-XH-A_1x02_P2.50mm_Vertical
- removed R9: 330, Resistor_SMD:R_0402_1005Metric
- removed U4: AMS1117-3.3, Package_TO_SOT_SMD:SOT-223-3_TabPin2
- added F1: 2920L050DR, Fuse:Fuse_2920_7451Metric, F.Cu at (126.0, 91.8)
- added JP3: Jumper_2_Bridged, Jumper:SolderJumper-2_P1.3mm_Bridged2Bar_RoundedPad1.0x1.5mm, F.Cu at (154.8, 94.5)
- added JP4: Jumper_3_Bridged12, Jumper:SolderJumper-3_P1.3mm_Bridged2Bar12_RoundedPad1.0x1.5mm, F.Cu at (151.5, 92.2)
- J10: footprint TerminalBlock_Phoenix:TerminalBlock_Phoenix_MKDS-1,5-2_1x02_P5.00mm_Horizontal -> _Local:1985807
- JP1: footprint Jumper:SolderJumper-2_P1.3mm_Bridged2Bar_Pad1.0x1.5mm -> Jumper:SolderJumper-2_P1.3mm_Bridged2Bar_RoundedPad1.0x1.5mm
- JP2: value Jumper_2_Bridged -> Jumper_3_Bridged12; footprint Jumper:SolderJumper-2_P1.3mm_Bridged2Bar_Pad1.0x1.5mm -> Jumper:SolderJumper-3_P1.3mm_Bridged2Bar12_RoundedPad1.0x1.5mm
- U1: value TSR_1-2450 -> TSR_1-2433
- moved IC1 50.2 mm to (169.2, 88.0)
- moved J9 48.3 mm to (144.8, 81.2), turned to 0 degrees
- moved R12 48.1 mm to (155.5, 81.0), turned to 0 degrees
- moved JP1 42.1 mm to (159.2, 94.5), turned to 180 degrees
- moved C9 41.6 mm to (126.1, 119.8), turned to 180 degrees
- moved U5 39.3 mm to (156.0, 86.2), turned to 90 degrees
- moved JP2 38.4 mm to (144.8, 90.0), turned to -90 degrees
- moved D5 27.5 mm to (155.2, 124.2), turned to -90 degrees
- moved SW1 26.5 mm to (171.0, 122.8), turned to 180 degrees
- moved R11 26.4 mm to (152.5, 86.2), turned to -90 degrees
- moved C1 26.0 mm to (146.8, 129.2), turned to -90 degrees
- moved R16 25.5 mm to (144.8, 124.7), turned to 90 degrees
- moved R13 24.0 mm to (146.0, 126.0), turned to -90 degrees
- moved D3 22.5 mm to (146.2, 123.5), turned to -90 degrees
- moved Q2 22.1 mm to (142.1, 124.7), turned to 180 degrees
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Connections:
- C7 pad 1: /BTN1 -> /TDI
- C8 pad 1: /BTN2 -> /TMS
- JP1 pad 1: /CAN_TX -> /DI
- JP1 pad 2: Net-(J11-Pad1) -> Net-(JP1-Pad2)
- JP2 pad 1: /CAN_RX -> /D(CTX)
- JP2 pad 2: Net-(J11-Pad2) -> /U1TXD
- Q1 pad 1: /LED1 -> /TDO
- Q2 pad 1: /LED2 -> /TCK
- R13 pad 2: /LED2 -> /TCK
- R14 pad 2: /LED1 -> /TDO
- R15 pad 1: /LED1 -> /TDO
- R16 pad 1: /LED2 -> /TCK
- R17 pad 1: /BTN1 -> /TDI
- R18 pad 1: /BTN2 -> /TMS
- U1 pad 3: +5V -> +3V3
- U2 pad 1: /U1RXD -> /RO
- U2 pad 4: /U1TXD -> /DI
- U5 pad 1: Net-(J11-Pad1) -> /D(CTX)
- U5 pad 4: Net-(J11-Pad2) -> /R(CRX)
- U6 pad 17: unconnected-(U6-Pad17) -> Net-(JP1-Pad2)
Routing:
- net +3V3: track 0.00 -> 147.3 mm, vias 0 -> 3
- net GND: track 0.00 -> 119.5 mm, vias 0 -> 14
- net /RESET: track 0.00 -> 64.9 mm, vias 0 -> 2
- net /RS(SCL): track 0.00 -> 51.4 mm
- net /SDO: track 0.00 -> 51.2 mm
- net /SDI(SDA): track 0.00 -> 50.9 mm
- net /CS: track 0.00 -> 48.0 mm, vias 0 -> 2
- net /WR(D/C): track 0.00 -> 46.8 mm, vias 0 -> 1
- net /IO0: track 0.00 -> 30.0 mm
- net Net-(BTNS1-Pad2): track 0.00 -> 25.8 mm
- net /485_DIR: track 0.00 -> 25.4 mm, vias 0 -> 2
- net /TCK: track 0.00 -> 24.4 mm
- net Net-(BTNS1-Pad1): track 0.00 -> 23.5 mm, vias 0 -> 2
- net /U1TXD: track 0.00 -> 22.9 mm, vias 0 -> 2
- net /CHIP_PU: track 0.00 -> 21.9 mm
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