File: UniversalControlPanel.kicad_pcb (KiCad board)
At the start: 2 copper layers, 70 x 55 mm, 53 parts, among them IC1 PSM712-LF-T7, J10 Conn_01x02, J3 Conn_01x40, J4 Conn_02x03_Odd_Even, J5 Conn_01x02, J8 Conn_01x07, J9 Conn_01x02, Q1 2N7002, Q2 2N7002, SW1 SW_Push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

Commit message: before reversing display
Parts:
- removed BTNS1: Conn_01x06, Connector_JST:JST_XH_B6B-XH-A_1x06_P2.50mm_Vertical
- removed J8: Conn_01x07, Connector_PinHeader_2.54mm:PinHeader_1x07_P2.54mm_Vertical
- added C10: 100n/16V, Capacitor_SMD:C_0402_1005Metric, F.Cu at (124.0, 106.5)
- added C11: 100n/16V, Capacitor_SMD:C_0402_1005Metric, F.Cu at (124.0, 111.3)
- added C3: 100n/16V, Capacitor_SMD:C_0402_1005Metric, F.Cu at (154.5, 89.2)
- added J1: Conn_01x09, Connector_JST:JST_XH_B9B-XH-A_1x09_P2.50mm_Vertical, F.Cu at (143.5, 129.8)
- added J2: Conn_01x09, Connector_PinHeader_2.54mm:PinHeader_1x09_P2.54mm_Vertical, F.Cu at (147.8, 115.0)
- added Q3: 2N7002, Package_TO_SOT_SMD:SOT-23, F.Cu at (125.5, 121.8)
- added R10: 15k, Resistor_SMD:R_0402_1005Metric, F.Cu at (132.5, 121.8)
- added R21: 8k2, Resistor_SMD:R_0402_1005Metric, F.Cu at (130.0, 124.5)
- added R22: 15k, Resistor_SMD:R_0402_1005Metric, F.Cu at (130.0, 121.8)
- added R9: 8k2, Resistor_SMD:R_0402_1005Metric, F.Cu at (132.5, 124.5)
- added U3: L78L05_SOT89, Package_TO_SOT_SMD:SOT-89-3, F.Cu at (133.0, 98.0)
- C4: value 100n -> 100n/16V
- J5: value Conn_01x02 -> Conn_01x03; footprint Connector_JST:JST_XH_B2B-XH-A_1x02_P2.50mm_Vertical -> Connector_JST:JST_XH_B3B-XH-A_1x03_P2.50mm_Vertical
- R4, R5, R6, R7: value R -> 68R
- moved C9 33.7 mm to (158.5, 129.0)
- moved R4 9.43 mm to (127.8, 118.8), turned to 90 degrees
- moved R5 7.36 mm to (126.5, 118.8), turned to -90 degrees
- moved R6 6.64 mm to (125.2, 118.8), turned to 90 degrees
- moved R7 5.64 mm to (124.0, 118.8), turned to -90 degrees
- moved JP2 4.81 mm to (149.0, 87.8), turned to 180 degrees
- moved D3 2.75 mm to (149.0, 123.5)
- moved D5 2.75 mm to (158.0, 124.2)
- moved Q1 2.75 mm to (153.8, 124.8)
- moved R13 2.75 mm to (148.8, 126.0)
- moved R14 2.75 mm to (157.0, 126.5)
- moved R15 2.75 mm to (156.5, 124.8)
- moved R16 2.75 mm to (147.6, 124.7)
- moved Q2 2.54 mm to (144.5, 124.0)
- moved J5 2.45 mm to (160.2, 81.2)
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Connections:
- C6 pad 1: Net-(C6-Pad1) -> /24V
- D4 pad 1: Net-(C6-Pad1) -> /24V
- F1 pad 1: /24V -> /IN_PWR
- F1 pad 2: Net-(C6-Pad1) -> /24V
- J10 pad 1: /24V -> /IN_PWR
- J3 pad 33: +5V -> /LEDA
- R4 pad 1: GND -> Net-(R7-Pad2)
- R5 pad 2: GND -> Net-(R7-Pad2)
- R6 pad 1: GND -> Net-(R7-Pad2)
- R7 pad 2: GND -> Net-(R7-Pad2)
- U1 pad 1: Net-(C6-Pad1) -> /24V
- U6 pad 14: unconnected-(U6-Pad14) -> Net-(R10-Pad1)
- U6 pad 15: unconnected-(U6-Pad15) -> Net-(R21-Pad2)
- U6 pad 16: unconnected-(U6-Pad16) -> /BLK
- U6 pad 24: unconnected-(U6-Pad24) -> Net-(U6-Pad24)
- U6 pad 25: /1WIRE -> /CS2
Routing:
- net GND: track 119.5 -> 208.5 mm, vias 14 -> 45
- net +3V3: track 147.3 -> 227.7 mm, vias 3 -> 9
- net /CTP-RST: track 0.00 -> 56.1 mm, vias 0 -> 4
- net /CTP-SDA: track 2.61 -> 54.8 mm, vias 1 -> 4
- net /CTP-SCL: track 4.04 -> 52.0 mm, vias 1 -> 4
- net /CTP-INT: track 4.01 -> 49.8 mm, vias 1 -> 4
- net /LEDA: track 0.00 -> 45.0 mm, vias 0 -> 3
- net Net-(R21-Pad2): track 0.00 -> 44.6 mm, vias 0 -> 2
- net Net-(R10-Pad1): track 0.00 -> 44.1 mm, vias 0 -> 2
- net Net-(U6-Pad24): track 0.00 -> 40.8 mm, vias 0 -> 2
- net /BLK: track 0.00 -> 35.4 mm, vias 0 -> 1
- net /DI: track 8.71 -> 30.9 mm, vias 2 -> 3
- net Net-(C6-Pad1): track 17.7 -> 0.00 mm
- net /24V: track 9.90 -> 20.0 mm
- net /IN_PWR: track 0.00 -> 9.90 mm
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- added copper zone on B.Cu, net GND
- added copper zone on F.Cu, net GND

Commit message: before upload
Parts:
- JP2, JP4: value Jumper_3_Bridged12 -> Jumper_2_Bridged; footprint Jumper:SolderJumper-3_P1.3mm_Bridged2Bar12_RoundedPad1.0x1.5mm -> Jumper:SolderJumper-2_P1.3mm_Bridged2Bar_RoundedPad1.0x1.5mm
- R4, R5, R6, R7: value 68R -> 75
- moved Q3 26.2 mm to (133.6, 96.8), turned to 180 degrees
- moved R7 23.3 mm to (124.2, 95.4), turned to 0 degrees
- moved R6 22.8 mm to (126.2, 96.0), turned to 180 degrees
- moved R5 22.3 mm to (128.2, 96.5), turned to 0 degrees
- moved R4 21.7 mm to (130.3, 97.2), turned to 180 degrees
- moved C11 18.5 mm to (136.1, 97.3), turned to 90 degrees
- moved U3 6.46 mm to (139.3, 96.6)
- moved C10 5.89 mm to (124.5, 112.4), turned to 90 degrees
- moved JP4 2.09 mm to (149.9, 90.8), turned to 180 degrees
- moved JP2 1.03 mm to (150.0, 88.1)
- moved R2 1.00 mm to (166.4, 99.2)
- moved R3 0.97 mm to (167.9, 99.2)
Connections:
- C11 pad 1: /LEDA -> /+5V
- J1 pad 8: /LEDA -> /+5V
- J2 pad 8: /BLK -> /RND
- J3 pad 10: unconnected-(J3-Pad10) -> /CTP-RST
- J3 pad 11: /WR(D/C) -> GND
- J3 pad 12: +3V3 -> GND
- J3 pad 13: /SDO -> GND
- J3 pad 2: /SDI(SDA) -> unconnected-(J3-Pad2)
- J3 pad 28: GND -> /SDO
- J3 pad 29: GND -> +3V3
- J3 pad 3: +3V3 -> unconnected-(J3-Pad3)
- J3 pad 30: GND -> /WR(D/C)
- J3 pad 31: /CTP-RST -> unconnected-(J3-Pad31)
- J3 pad 32: /CTP-SDA -> /CS
- J3 pad 33: /LEDA -> /RS(SCL)
- J3 pad 34: /LEDK1 -> /RESET
- J3 pad 35: /LEDK2 -> /CTP-SCL
- J3 pad 36: /LEDK3 -> /CTP-INT
- J3 pad 37: /LEDK4 -> unconnected-(J3-Pad37)
- J3 pad 38: unconnected-(J3-Pad38) -> +3V3
- J3 pad 39: unconnected-(J3-Pad39) -> /SDI(SDA)
- J3 pad 4: unconnected-(J3-Pad4) -> /LEDK4
- J3 pad 5: /CTP-INT -> /LEDK3
- J3 pad 6: /CTP-SCL -> /LEDK2
- J3 pad 7: /RESET -> /LEDK1
- J3 pad 8: /RS(SCL) -> /+5V
- J3 pad 9: /CS -> /CTP-SDA
- Q3 pad 1: Net-(U6-Pad24) -> /BLK
- U3 pad 1: /LEDA -> /+5V
- U6 pad 16: /BLK -> /RND
- U6 pad 24: Net-(U6-Pad24) -> unconnected-(U6-Pad24)
- U6 pad 4: unconnected-(U6-Pad4) -> /BLK
Routing:
- net /+5V: track 0.00 -> 68.6 mm, vias 0 -> 2
- net /LEDA: track 45.0 -> 0.00 mm, vias 3 -> 0
- net Net-(U6-Pad24): track 40.8 -> 0.00 mm, vias 2 -> 0
- net /RND: track 0.00 -> 34.9 mm, vias 0 -> 3
- net GND: track 208.5 -> 232.1 mm, vias 45 -> 56
- net /DI: track 30.9 -> 8.63 mm, vias 3 -> 0
- net /RESET: track 64.4 -> 49.8 mm, vias 1 -> 0
- net /CTP-INT: track 49.8 -> 61.9 mm
- net /BLK: track 35.4 -> 46.3 mm, vias 1 -> 2
- net /CTP-SCL: track 52.0 -> 60.3 mm
- net /SDI(SDA): track 50.9 -> 42.9 mm, vias 0 -> 1
- net /RO: track 14.2 -> 8.80 mm
- net /CS: track 46.2 -> 41.3 mm, vias 2 -> 0
- net /485_DIR: track 27.7 -> 32.6 mm
- net /RS(SCL): track 50.1 -> 45.5 mm
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Other:
- board text added: "1"
- board text added: "40"
